Commit message: Added hugin CAD for visualization

File: real_auv/hugin_description/urdf/hugin_auv_base.urdf.xacro (robot description, xacro)
@@ -3,13 +3,13 @@
   <!-- Properties -->
   <xacro:property name="M_PI" value="3.14159" />
-  <!-- <xacro:property name="visual_mesh_file" value="file://$(find hugin_description)/mesh/hugin_body.dae"/> -->
+  <xacro:property name="visual_mesh_file" value="file://$(find hugin_description)/mesh/hugin_body.dae"/>
   <xacro:macro name="hugin_auv_base" params="namespace debug">
     <link name="${namespace}/base_link">
-<!--       <visual>
+      <visual>
         <origin xyz="0 0 0" rpy="0 0 0"/>
         <geometry>
           <mesh filename="${visual_mesh_file}" scale="3 3 3" />
         </geometry>
-      </visual> -->
+      </visual>
 <!--       <collision>
         <origin xyz="0 0 0" rpy="0 ${0.5*pi} 0"/>

Commit message: Added actual Hugin model, just for visualization

File: real_auv/hugin_description/urdf/hugin_auv_base.urdf.xacro (robot description, xacro)
@@ -3,5 +3,8 @@
   <!-- Properties -->
   <xacro:property name="M_PI" value="3.14159" />
-  <xacro:property name="visual_mesh_file" value="file://$(find hugin_description)/mesh/hugin_body.dae"/>
+  <xacro:property name="visual_mesh_file" value="file://$(find hugin_description)/mesh/Hugin_big_meter.dae"/>
+ <material name="blue">
+    <color rgba="0 0 0.8 1"/>
+  </material>
   <xacro:macro name="hugin_auv_base" params="namespace debug">
     <link name="${namespace}/base_link">
@@ -9,6 +12,7 @@
         <origin xyz="0 0 0" rpy="0 0 0"/>
         <geometry>
-          <mesh filename="${visual_mesh_file}" scale="3 3 3" />
+          <mesh filename="${visual_mesh_file}" scale="0.001 0.001 0.001" />
         </geometry>
+        <material name="blue"/>
       </visual>
 <!--       <collision>

Commit message: Simplified hugin model with color

File: real_auv/hugin_description/urdf/hugin_auv_base.urdf.xacro (robot description, xacro)
@@ -3,5 +3,5 @@
   <!-- Properties -->
   <xacro:property name="M_PI" value="3.14159" />
-  <xacro:property name="visual_mesh_file" value="file://$(find hugin_description)/mesh/Hugin_big_meter.dae"/>
+  <xacro:property name="visual_mesh_file" value="file://$(find hugin_description)/mesh/hugin_color.dae"/>
  <material name="blue">
     <color rgba="0 0 0.8 1"/>

Commit message: Moved MBES pose within Hugin

File: real_auv/hugin_description/urdf/hugin_auv_base.urdf.xacro (robot description, xacro)
@@ -31,5 +31,5 @@
     </link>
     <joint name="${namespace}/mbes_joint" type="fixed">
-      <origin xyz="5.0 0.0 0.0" rpy="0 ${M_PI} 0" />
+      <origin xyz="2.0 0.0 0.0" rpy="0 ${M_PI} 0" />
       <parent link="${namespace}/base_link"/>
       <child link="${namespace}/mbes_link"/>

Commit message: MBES config for the MMT Ping

File: real_auv/hugin_description/urdf/hugin_auv_base.urdf.xacro (robot description, xacro)
@@ -31,5 +31,6 @@
     </link>
     <joint name="${namespace}/mbes_joint" type="fixed">
-      <origin xyz="2.0 0.0 0.0" rpy="0 ${M_PI} 0" />
+      <!-- <origin xyz="4.0 0.0 0.0" rpy="0.43 ${M_PI} 0" /> --> <!-- Ping in lost_targets -->
+      <origin xyz="4.0 0.0 0.0" rpy="0.43 ${M_PI} 0" />
       <parent link="${namespace}/base_link"/>
       <child link="${namespace}/mbes_link"/>

Commit message: Option to fix Hugin visual for Ping surveys

File: real_auv/hugin_description/urdf/hugin_auv_base.urdf.xacro (robot description, xacro)
@@ -10,4 +10,5 @@
     <link name="${namespace}/base_link">
       <visual>
+        <!-- <origin xyz="0 -10.0 0" rpy="0 0 0"/> --> <!-- To trick the eye with Hugin on Ping survey -->
         <origin xyz="0 0 0" rpy="0 0 0"/>
         <geometry>

Commit message: Added start/stop ping to replay parts of missions as params. Fixed pings on PF

File: real_auv/hugin_description/urdf/hugin_auv_base.urdf.xacro (robot description, xacro)
@@ -33,5 +33,5 @@
     <joint name="${namespace}/mbes_joint" type="fixed">
       <!-- <origin xyz="4.0 0.0 0.0" rpy="0.43 ${M_PI} 0" /> --> <!-- Ping in lost_targets -->
-      <origin xyz="4.0 0.0 0.0" rpy="0.43 ${M_PI} 0" />
+      <origin xyz="4. 0. 0.0" rpy="0.43 ${M_PI} 0" />
       <parent link="${namespace}/base_link"/>
       <child link="${namespace}/mbes_link"/>

Commit message: MBES tf back to normal for Hugin

File: real_auv/hugin_description/urdf/hugin_auv_base.urdf.xacro (robot description, xacro)
@@ -33,5 +33,5 @@
     <joint name="${namespace}/mbes_joint" type="fixed">
       <!-- <origin xyz="4.0 0.0 0.0" rpy="0.43 ${M_PI} 0" /> --> <!-- Ping in lost_targets -->
-      <origin xyz="4. 0. 0.0" rpy="0.43 ${M_PI} 0" />
+      <origin xyz="0. 0. 0.0" rpy="0.0 ${M_PI} 0" />
       <parent link="${namespace}/base_link"/>
       <child link="${namespace}/mbes_link"/>

Commit message: GP sampling and ray-tracing running and tested. The mbes frame has x axis now like the base

File: real_auv/hugin_description/urdf/hugin_auv_base.urdf.xacro (robot description, xacro)
@@ -33,5 +33,5 @@
     <joint name="${namespace}/mbes_joint" type="fixed">
       <!-- <origin xyz="4.0 0.0 0.0" rpy="0.43 ${M_PI} 0" /> --> <!-- Ping in lost_targets -->
-      <origin xyz="0. 0. 0.0" rpy="0.0 ${M_PI} 0" />
+      <origin xyz="0. 0. 0.0" rpy="${M_PI} 0.0 0.0" />
       <parent link="${namespace}/base_link"/>
       <child link="${namespace}/mbes_link"/>

Commit message: Real MBES beams in same order than GPs. MBES frame from tf used. GP-PF running with real data on lost_targets

File: real_auv/hugin_description/urdf/hugin_auv_base.urdf.xacro (robot description, xacro)
@@ -32,6 +32,6 @@
     </link>
     <joint name="${namespace}/mbes_joint" type="fixed">
-      <!-- <origin xyz="4.0 0.0 0.0" rpy="0.43 ${M_PI} 0" /> --> <!-- Ping in lost_targets -->
-      <origin xyz="0. 0. 0.0" rpy="${M_PI} 0.0 0.0" />
+      <origin xyz="4.0 0.0 0.0" rpy="${M_PI - 0.38} 0 0" /> <!-- Ping in lost_targets -->
+      <!-- <origin xyz="0. 0. 0.0" rpy="${M_PI} 0.0 0.0" /> -->
       <parent link="${namespace}/base_link"/>
       <child link="${namespace}/mbes_link"/>

Commit message: Now both real and sim data can be used without changes in the scripts

File: real_auv/hugin_description/urdf/hugin_auv_base.urdf.xacro (robot description, xacro)
@@ -32,5 +32,5 @@
     </link>
     <joint name="${namespace}/mbes_joint" type="fixed">
-      <origin xyz="4.0 0.0 0.0" rpy="${M_PI - 0.38} 0 0" /> <!-- Ping in lost_targets -->
+      <origin xyz="4.0 0.0 0.0" rpy="${M_PI - 0.38} 0 0" /> Ping in lost_targets
       <!-- <origin xyz="0. 0. 0.0" rpy="${M_PI} 0.0 0.0" /> -->
       <parent link="${namespace}/base_link"/>

Commit message: Now z in map frames used instead of ping ranges. PF with IGL working both on GT and sim.

File: real_auv/hugin_description/urdf/hugin_auv_base.urdf.xacro (robot description, xacro)
@@ -32,5 +32,6 @@
     </link>
     <joint name="${namespace}/mbes_joint" type="fixed">
-      <origin xyz="4.0 0.0 0.0" rpy="${M_PI - 0.38} 0 0" /> Ping in lost_targets
+      <!--Ping in lost_targets-->
+      <origin xyz="4.0 0.0 0.0" rpy="${M_PI - 0.38} 0 0" />
       <!-- <origin xyz="0. 0. 0.0" rpy="${M_PI} 0.0 0.0" /> -->
       <parent link="${namespace}/base_link"/>

Commit message: IGL PF running on overnight2020

File: real_auv/hugin_description/urdf/hugin_auv_base.urdf.xacro (robot description, xacro)
@@ -33,6 +33,6 @@
     <joint name="${namespace}/mbes_joint" type="fixed">
       <!--Ping in lost_targets-->
-      <origin xyz="4.0 0.0 0.0" rpy="${M_PI - 0.38} 0 0" />
-      <!-- <origin xyz="0. 0. 0.0" rpy="${M_PI} 0.0 0.0" /> -->
+      <!-- <origin xyz="4.0 0.0 0.0" rpy="${M_PI - 0.38} 0 0" />  -->
+      <origin xyz="3.5 0. 0.0" rpy="0.0 0.0 0.0" />
       <parent link="${namespace}/base_link"/>
       <child link="${namespace}/mbes_link"/>

Commit message: Adjusted mbes tf from real Hugin

File: real_auv/hugin_description/urdf/hugin_auv_base.urdf.xacro (robot description, xacro)
@@ -34,5 +34,5 @@
       <!--Ping in lost_targets-->
       <!-- <origin xyz="4.0 0.0 0.0" rpy="${M_PI - 0.38} 0 0" />  -->
-      <origin xyz="3.5 0. 0.0" rpy="0.0 0.0 0.0" />
+      <origin xyz="3.5 0. -0.70" rpy="0.0 0.0 0.0" />
       <parent link="${namespace}/base_link"/>
       <child link="${namespace}/mbes_link"/>

Commit message: MBES frame on top of base_link for now

File: real_auv/hugin_description/urdf/hugin_auv_base.urdf.xacro (robot description, xacro)
@@ -34,5 +34,5 @@
       <!--Ping in lost_targets-->
       <!-- <origin xyz="4.0 0.0 0.0" rpy="${M_PI - 0.38} 0 0" />  -->
-      <origin xyz="3.5 0. -0.70" rpy="0.0 0.0 0.0" />
+      <origin xyz="0.0 0. -0.00" rpy="0.0 0.0 0.0" />
       <parent link="${namespace}/base_link"/>
       <child link="${namespace}/mbes_link"/>

Commit message: Several particles training several GPs tested

File: real_auv/hugin_description/urdf/hugin_auv_base.urdf.xacro (robot description, xacro)
@@ -34,5 +34,5 @@
       <!--Ping in lost_targets-->
       <!-- <origin xyz="4.0 0.0 0.0" rpy="${M_PI - 0.38} 0 0" />  -->
-      <origin xyz="3.5 0. -0.70" rpy="0.0 0.0 0.0" />
+      <origin xyz="0.0 0.0 0.0" rpy="0.0 0.0 0.0" />
       <parent link="${namespace}/base_link"/>
       <child link="${namespace}/mbes_link"/>

Commit message: Getting remo with ripples dataset running

File: real_auv/hugin_description/urdf/hugin_auv_base.urdf.xacro (robot description, xacro)
@@ -10,5 +10,4 @@
     <link name="${namespace}/base_link">
       <visual>
-        <!-- <origin xyz="0 -10.0 0" rpy="0 0 0"/> --> <!-- To trick the eye with Hugin on Ping survey -->
         <origin xyz="0 0 0" rpy="0 0 0"/>
         <geometry>
@@ -34,5 +33,5 @@
       <!--Ping in lost_targets-->
       <!-- <origin xyz="4.0 0.0 0.0" rpy="${M_PI - 0.38} 0 0" />  -->
-      <origin xyz="0.0 0.0 0.0" rpy="0.0 0.0 0.0" />
+      <origin xyz="-10.0 0.0 0.0" rpy="0.0 0.0 0.0" />  <!-- MBES for ripples -->
       <parent link="${namespace}/base_link"/>
       <child link="${namespace}/mbes_link"/>

Commit message: [JXRBPF] Adapted the RBPF to work on the Xavier

File: real_auv/hugin_description/urdf/hugin_auv_base.urdf.xacro (robot description, xacro)
@@ -10,4 +10,5 @@
     <link name="${namespace}/base_link">
       <visual>
+        <!-- <origin xyz="0 -10.0 0" rpy="0 0 0"/> --> <!-- To trick the eye with Hugin on Ping survey -->
         <origin xyz="0 0 0" rpy="0 0 0"/>
         <geometry>
@@ -16,22 +17,9 @@
         <material name="blue"/>
       </visual>
-<!--       <collision>
-        <origin xyz="0 0 0" rpy="0 ${0.5*pi} 0"/>
-        <geometry>
-          <cylinder length="${length}" radius="${radius}"/>
-        </geometry>
-      </collision>
-      <inertial>
-        <mass value="${mass}" />
-        <origin xyz="${com}" rpy="0 0 0"/>
-        <inertia ixx="0.0294" ixy="0" ixz="0"
-                 iyy="1.6202" iyz="0"
-                 izz="1.6202" />
-      </inertial> -->
     </link>
     <joint name="${namespace}/mbes_joint" type="fixed">
       <!--Ping in lost_targets-->
       <!-- <origin xyz="4.0 0.0 0.0" rpy="${M_PI - 0.38} 0 0" />  -->
-      <origin xyz="-10.0 0.0 0.0" rpy="0.0 0.0 0.0" />  <!-- MBES for ripples -->
+      <origin xyz="0.0 0.0 0.0" rpy="0.0 0.0 0.0" />
       <parent link="${namespace}/base_link"/>
       <child link="${namespace}/mbes_link"/>

Commit message: Got the parallel particles running

File: real_auv/hugin_description/urdf/hugin_auv_base.urdf.xacro (robot description, xacro)
@@ -33,5 +33,5 @@
       <!--Ping in lost_targets-->
       <!-- <origin xyz="4.0 0.0 0.0" rpy="${M_PI - 0.38} 0 0" />  -->
-      <origin xyz="-10.0 0.0 0.0" rpy="0.0 0.0 0.0" />  <!-- MBES for ripples -->
+      <origin xyz="0.0 0.0 0.0" rpy="0.0 0.0 0.0" />  <!-- MBES for ripples -->
       <parent link="${namespace}/base_link"/>
       <child link="${namespace}/mbes_link"/>

Commit message: Added SSS link to Hugin

File: real_auv/hugin_description/urdf/hugin_auv_base.urdf.xacro (robot description, xacro)
@@ -57,4 +57,29 @@
       </collision>
     </link>
+    <joint name="${namespace}/sss_joint" type="fixed">
+      <origin xyz="0.0 0.0 0.0" rpy="0.0 0.0 0.0" />
+      <parent link="${namespace}/base_link"/>
+      <child link="${namespace}/sss_link"/>
+    </joint>
+    <link name="${namespace}/sss_link">
+      <inertial>
+        <mass value="0.001"/>
+        <origin rpy="0 0 0" xyz="0 0 0"/>
+        <inertia ixx="0.0001" ixy="0" ixz="0" iyy="0.000001" iyz="0" izz="0.0001"/>
+      </inertial>
+      <visual>
+        <origin rpy="0 0 0" xyz="0 0 0"/>
+        <geometry>
+          <box size="0.01 0.01 0.01"/>
+        </geometry>
+        <material name="blue"/>
+      </visual>
+      <collision>
+        <origin rpy="0 0 0" xyz="0 0 0"/>
+        <geometry>
+          <box size="0.01 0.01 0.01"/>
+        </geometry>
+      </collision>
+    </link>
   </xacro:macro>
 </robot>
